File: h_bridge.sch (KiCad schematic (older format))
At the start: 11 parts, among them Q1 PSMN5R2-60YL, Q2 PSMN5R2-60YL, Q3 PSMN5R2-60YL, Q4 PSMN5R2-60YL

Commit message: basic h-bridge schematic
Parts:
- removed R1: R, Resistor_SMD:R_0603_1608Metric, symbol Device:R
Connections:
- net labels added: +BATT, GNDPWR
- net labels removed: GND, V_motor
- wire segments 41 -> 42
Changed lines of the file:
@@
 EESchema Schematic File Version 4
-LIBS:motor-controller-v8-cache
-EELAYER 26 0
+EELAYER 30 0
 EELAYER END
 $Descr A4 11693 8268
@@
 	4900 2850 4900 2750
 Wire Wire Line
-	4900 2750 6150 2750
+	4900 2750 5500 2750
 Wire Wire Line
 	6150 2750 6150 2850
@@
 AR Path="/5C7CBEEA/5C896002" Ref="D1"  Part="1"
 AR Path="/5C7CEE9C/5C896002" Ref="D7"  Part="1"
-F 0 "D7" V 4404 3329 50  0000 L CNN
+AR Path="/5E6C9798/5E6D3963/5C896002" Ref="D3"  Part="1"
+AR Path="/5E6D5B01/5E6D3963/5C896002" Ref="D?"  Part="1"
+AR Path="/5E6D6147/5E6D3963/5C896002" Ref="D11"  Part="1"
+F 0 "D3" V 4404 3329 50  0000 L CNN
 F 1 "D_TVS" V 4495 3329 50  0000 L CNN
 F 2 "Diode_SMD:D_0805_2012Metric" H 4450 3250 50  0001 C CNN
@@
 AR Path="/5C7CBEEA/5C896003" Ref="D2"  Part="1"
 AR Path="/5C7CEE9C/5C896003" Ref="D8"  Part="1"
-F 0 "D8" V 4404 3979 50  0000 L CNN
+AR Path="/5E6C9798/5E6D3963/5C896003" Ref="D4"  Part="1"
+AR Path="/5E6D5B01/5E6D3963/5C896003" Ref="D?"  Part="1"
+AR Path="/5E6D6147/5E6D3963/5C896003" Ref="D12"  Part="1"
+F 0 "D4" V 4404 3979 50  0000 L CNN
 F 1 "D_TVS" V 4495 3979 50  0000 L CNN
 F 2 "Diode_SMD:D_0805_2012Metric" H 4450 3900 50  0001 C CNN
@@
 AR Path="/5C7CBEEA/5C896004" Ref="D6"  Part="1"
 AR Path="/5C7CEE9C/5C896004" Ref="D12"  Part="1"
-F 0 "D12" V 6504 3979 50  0000 L CNN
+AR Path="/5E6C9798/5E6D3963/5C896004" Ref="D8"  Part="1"
+AR Path="/5E6D5B01/5E6D3963/5C896004" Ref="D?"  Part="1"
+AR Path="/5E6D6147/5E6D3963/5C896004" Ref="D16"  Part="1"
+F 0 "D8" V 6504 3979 50  0000 L CNN
 F 1 "D_TVS" V 6595 3979 50  0000 L CNN
 F 2 "Diode_SMD:D_0805_2012Metric" H 6550 3900 50  0001 C CNN
@@
 AR Path="/5C7CBEEA/5C896005" Ref="D5"  Part="1"
 AR Path="/5C7CEE9C/5C896005" Ref="D11"  Part="1"
-F 0 "D11" V 6504 3329 50  0000 L CNN
+AR Path="/5E6C9798/5E6D3963/5C896005" Ref="D7"  Part="1"
+AR Path="/5E6D5B01/5E6D3963/5C896005" Ref="D?"  Part="1"
+AR Path="/5E6D6147/5E6D3963/5C896005" Ref="D15"  Part="1"
+F 0 "D7" V 6504 3329 50  0000 L CNN
 F 1 "D_TVS" V 6595 3329 50  0000 L CNN
 F 2 "Diode_SMD:D_0805_2012Metric" H 6550 3250 50  0001 C CNN
@@
 AR Path="/5C7CBEEA/5C896006" Ref="D3"  Part="1"
 AR Path="/5C7CEE9C/5C896006" Ref="D9"  Part="1"
-F 0 "D9" V 5304 3779 50  0000 L CNN
+AR Path="/5E6C9798/5E6D3963/5C896006" Ref="D5"  Part="1"
+AR Path="/5E6D5B01/5E6D3963/5C896006" Ref="D?"  Part="1"
+AR Path="/5E6D6147/5E6D3963/5C896006" Ref="D13"  Part="1"
+F 0 "D5" V 5304 3779 50  0000 L CNN
 F 1 "D_TVS" V 5395 3779 50  0000 L CNN
 F 2 "Diode_SMD:D_0805_2012Metric" H 5350 3700 50  0001 C CNN
@@
 AR Path="/5C7CBEEA/5C896007" Ref="D4"  Part="1"
 AR Path="/5C7CEE9C/5C896007" Ref="D10"  Part="1"
-F 0 "D10" V 5654 3779 50  0000 L CNN
+AR Path="/5E6C9798/5E6D3963/5C896007" Ref="D6"  Part="1"
+AR Path="/5E6D5B01/5E6D3963/5C896007" Ref="D?"  Part="1"
+AR Path="/5E6D6147/5E6D3963/5C896007" Ref="D14"  Part="1"
+F 0 "D6" V 5654 3779 50  0000 L CNN
 F 1 "D_TVS" V 5745 3779 50  0000 L CNN
 F 2 "Diode_SMD:D_0805_2012Metric" H 5700 3700 50  0001 C CNN
@@
 Wire Wire Line
 	5700 3400 6150 3400
-Text Label 5350 2750 0    50   ~ 0
-V_motor
 Text Label 5250 4050 0    50   ~ 0
 H_bridge_bot
@@
 Text Label 4350 3700 0    50   ~ 0
 GHA1
-$Comp
-L Device:R R?
-U 1 1 5C896008
-P 5550 4300
-AR Path="/5C896008" Ref="R?"  Part="1"
-AR Path="/5C7CBEEA/5C896008" Ref="R1"  Part="1"
-AR Path="/5C7CEE9C/5C896008" Ref="R2"  Part="1"
-F 0 "R2" H 5620 4346 50  0000 L CNN
-F 1 "R" H 5620 4255 50  0000 L CNN
-F 2 "Resistor_SMD:R_0603_1608Metric" V 5480 4300 50  0001 C CNN
-F 3 "~" H 5550 4300 50  0001 C CNN
-	1    5550 4300
-	1    0    0    -1
-$EndComp
-Wire Wire Line
-	5550 4150 5550 4050
 Connection ~ 5550 4050
 Wire Wire Line
 	5550 4050 5700 4050
-$Comp
-L power:GND #PWR?
-U 1 1 5C896009
-P 5550 4550
-AR Path="/5C896009" Ref="#PWR?"  Part="1"
-AR Path="/5C7CBEEA/5C896009" Ref="#PWR0101"  Part="1"
-AR Path="/5C7CEE9C/5C896009" Ref="#PWR0102"  Part="1"
-F 0 "#PWR0102" H 5550 4300 50  0001 C CNN
-F 1 "GND" H 5555 4377 50  0000 C CNN
-F 2 "" H 5550 4550 50  0001 C CNN
-F 3 "" H 5550 4550 50  0001 C CNN
-	1    5550 4550
-	1    0    0    -1
-$EndComp
-Wire Wire Line
-	5550 4450 5550 4550
 Text HLabel 4300 3050 0    50   Input ~ 0
 GHA1
@@
 AR Path="/5C7CBEEA/5C7DFA52" Ref="Q1"  Part="1"
 AR Path="/5C7CEE9C/5C7DFA52" Ref="Q5"  Part="1"
-F 0 "Q5" H 5006 3096 50  0000 L CNN
+AR Path="/5E6C9798/5E6D3963/5C7DFA52" Ref="Q1"  Part="1"
+AR Path="/5E6D5B01/5E6D3963/5C7DFA52" Ref="Q?"  Part="1"
+AR Path="/5E6D6147/5E6D3963/5C7DFA52" Ref="Q5"  Part="1"
+F 0 "Q1" H 5006 3096 50  0000 L CNN
 F 1 "PSMN5R2-60YL" H 5006 3005 50  0000 L CNN
 F 2 "Package_TO_SOT_SMD:LFPAK56" H 4950 3050 50  0001 C CNN
@@
 AR Path="/5C7CBEEA/5C7DFAA0" Ref="Q2"  Part="1"
 AR Path="/5C7CEE9C/5C7DFAA0" Ref="Q6"  Part="1"
-F 0 "Q6" H 5006 3746 50  0000 L CNN
+AR Path="/5E6C9798/5E6D3963/5C7DFAA0" Ref="Q2"  Part="1"
+AR Path="/5E6D5B01/5E6D3963/5C7DFAA0" Ref="Q?"  Part="1"
+AR Path="/5E6D6147/5E6D3963/5C7DFAA0" Ref="Q6"  Part="1"
+F 0 "Q2" H 5006 3746 50  0000 L CNN
 F 1 "PSMN5R2-60YL" H 5006 3655 50  0000 L CNN
 F 2 "Package_TO_SOT_SMD:LFPAK56" H 4950 3700 50  0001 C CNN
@@
 AR Path="/5C7CBEEA/5C7DFAE0" Ref="Q3"  Part="1"
 AR Path="/5C7CEE9C/5C7DFAE0" Ref="Q7"  Part="1"
-F 0 "Q7" H 6456 3096 50  0000 L CNN
+AR Path="/5E6C9798/5E6D3963/5C7DFAE0" Ref="Q3"  Part="1"
+AR Path="/5E6D5B01/5E6D3963/5C7DFAE0" Ref="Q?"  Part="1"
+AR Path="/5E6D6147/5E6D3963/5C7DFAE0" Ref="Q7"  Part="1"
+F 0 "Q3" H 6456 3096 50  0000 L CNN
 F 1 "PSMN5R2-60YL" H 6456 3005 50  0000 L CNN
 F 2 "Package_TO_SOT_SMD:LFPAK56" H 6400 3050 50  0001 C CNN
@@
 AR Path="/5C7CBEEA/5C7E0276" Ref="Q4"  Part="1"
 AR Path="/5C7CEE9C/5C7E0276" Ref="Q8"  Part="1"
-F 0 "Q8" H 6456 3746 50  0000 L CNN
+AR Path="/5E6C9798/5E6D3963/5C7E0276" Ref="Q4"  Part="1"
+AR Path="/5E6D5B01/5E6D3963/5C7E0276" Ref="Q?"  Part="1"
+AR Path="/5E6D6147/5E6D3963/5C7E0276" Ref="Q8"  Part="1"
+F 0 "Q4" H 6456 3746 50  0000 L CNN
 F 1 "PSMN5R2-60YL" H 6456 3655 50  0000 L CNN
 F 2 "Package_TO_SOT_SMD:LFPAK56" H 6400 3700 50  0001 C CNN
@@
 	-1   0    0    -1
 $EndComp
+$Comp
+L power:GNDPWR #PWR0110
+U 1 1 5E6A018B
+P 5550 4250
+AR Path="/5C7CEE9C/5E6A018B" Ref="#PWR0110"  Part="1"
+AR Path="/5C7CBEEA/5E6A018B" Ref="#PWR0109"  Part="1"
+AR Path="/5E6C9798/5E6D3963/5E6A018B" Ref="#PWR0109"  Part="1"
+AR Path="/5E6D5B01/5E6D3963/5E6A018B" Ref="#PWR?"  Part="1"
+AR Path="/5E6D6147/5E6D3963/5E6A018B" Ref="#PWR0118"  Part="1"
+F 0 "#PWR0109" H 5550 4050 50  0001 C CNN
+F 1 "GNDPWR" H 5554 4096 50  0000 C CNN
+F 2 "" H 5550 4200 50  0001 C CNN
+F 3 "" H 5550 4200 50  0001 C CNN
+	1    5550 4250
+	1    0    0    -1
+$EndComp
+$Comp
+L power:+BATT #PWR0112
+U 1 1 5E69D2AF
+P 5500 2650
+F 0 "#PWR0112" H 5500 2500 50  0001 C CNN
+F 1 "+BATT" H 5515 2823 50  0000 C CNN
+F 2 "" H 5500 2650 50  0001 C CNN
+F 3 "" H 5500 2650 50  0001 C CNN
+	1    5500 2650
+	1    0    0    -1
+$EndComp
+Wire Wire Line
+	5500 2650 5500 2750
+Connection ~ 5500 2750
+Wire Wire Line
+	5500 2750 6150 2750
+Wire Wire Line
+	5550 4050 5550 4250
 $EndSCHEMATC
