File: motor-controller-v8.kicad_pcb (KiCad board)
At the start: 2 copper layers, 30 parts, among them J1 Conn_01x02, J2 Conn_01x02, Q1 PSMN5R2-60YL, Q2 PSMN5R2-60YL, Q3 PSMN5R2-60YL, Q4 PSMN5R2-60YL, Q5 PSMN5R2-60YL, Q6 PSMN5R2-60YL, Q7 PSMN5R2-60YL, Q8 PSMN5R2-60YL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

Commit message: basic h-bridge schematic
Parts:
- removed D1, D10, D11, D12, D2, D3, D4, D5, D6, D7, D8, D9: D_TVS, Diode_SMD:D_0805_2012Metric
- removed J1, J2: Conn_01x02, Connector_PinHeader_2.54mm:PinHeader_1x02_P2.54mm_Vertical
- removed Q1, Q2, Q3, Q4, Q5, Q6, Q7, Q8: PSMN5R2-60YL, Package_TO_SOT_SMD:LFPAK56
- removed R1, R2: R, Resistor_SMD:R_0603_1608Metric
- removed U1: TM4C1230H6PM, Package_QFP:LQFP-64_10x10mm_P0.5mm
- removed U2: ET60T-02-24-02-X-RTX-GP, Exodus_Connectors:ET60T-02-24-02-X-RTX-GP-HS
- removed U3: HIP4080A, Package_QFP:LQFP-64_10x10mm_P0.5mm
- removed U4: HIP4080A, Package_SO:SOIC-16_3.9x9.9mm_P1.27mm
- removed U5, U6: LTC4364HS, Package_SO:SOIC-16_3.9x9.9mm_P1.27mm
Routing:
- net /h_bridge/H_bridge_bot: track 10.6 -> 0.00 mm
- net /h_bridge/MOTOR+: track 10.2 -> 0.00 mm
- net /h_bridge/GHA1: track 9.99 -> 0.00 mm
- net /h_bridge/GHA2: track 9.68 -> 0.00 mm
- net /h_bridge/MOTOR-: track 7.93 -> 0.00 mm
