File: h-bridge-demo/h_bridge.sch (KiCad schematic (older format))
At the start: 10 parts, among them Q1 PSMN5R2-60YL, Q2 PSMN5R2-60YL, Q3 PSMN5R2-60YL, Q4 PSMN5R2-60YL

Commit message: adding pwm isolation
Parts:
- D1, D2, D5, D6: footprint Diode_SMD:D_0805_2012Metric -> Diode_SMD:D_SMA
- D3, D4: footprint Diode_SMD:D_0805_2012Metric -> Diode_SMD:D_SMB
Changed lines of the file:
@@
 EESchema Schematic File Version 4
+LIBS:motor-controller-v8-cache
 EELAYER 30 0
 EELAYER END
@@
 F 0 "D3" V 4404 3329 50  0000 L CNN
 F 1 "D_TVS" V 4495 3329 50  0000 L CNN
-F 2 "Diode_SMD:D_0805_2012Metric" H 4450 3250 50  0001 C CNN
+F 2 "Diode_SMD:D_SMA" H 4450 3250 50  0001 C CNN
 F 3 "~" H 4450 3250 50  0001 C CNN
 	1    4450 3250
@@
 F 0 "D4" V 4404 3979 50  0000 L CNN
 F 1 "D_TVS" V 4495 3979 50  0000 L CNN
-F 2 "Diode_SMD:D_0805_2012Metric" H 4450 3900 50  0001 C CNN
+F 2 "Diode_SMD:D_SMA" H 4450 3900 50  0001 C CNN
 F 3 "~" H 4450 3900 50  0001 C CNN
 	1    4450 3900
@@
 F 0 "D8" V 6504 3979 50  0000 L CNN
 F 1 "D_TVS" V 6595 3979 50  0000 L CNN
-F 2 "Diode_SMD:D_0805_2012Metric" H 6550 3900 50  0001 C CNN
+F 2 "Diode_SMD:D_SMA" H 6550 3900 50  0001 C CNN
 F 3 "~" H 6550 3900 50  0001 C CNN
 	1    6550 3900
@@
 F 0 "D7" V 6504 3329 50  0000 L CNN
 F 1 "D_TVS" V 6595 3329 50  0000 L CNN
-F 2 "Diode_SMD:D_0805_2012Metric" H 6550 3250 50  0001 C CNN
+F 2 "Diode_SMD:D_SMA" H 6550 3250 50  0001 C CNN
 F 3 "~" H 6550 3250 50  0001 C CNN
 	1    6550 3250
@@
 F 0 "D5" V 5304 3779 50  0000 L CNN
 F 1 "D_TVS" V 5395 3779 50  0000 L CNN
-F 2 "Diode_SMD:D_0805_2012Metric" H 5350 3700 50  0001 C CNN
+F 2 "Diode_SMD:D_SMB" H 5350 3700 50  0001 C CNN
 F 3 "~" H 5350 3700 50  0001 C CNN
 	1    5350 3700
@@
 F 0 "D6" V 5654 3779 50  0000 L CNN
 F 1 "D_TVS" V 5745 3779 50  0000 L CNN
-F 2 "Diode_SMD:D_0805_2012Metric" H 5700 3700 50  0001 C CNN
+F 2 "Diode_SMD:D_SMB" H 5700 3700 50  0001 C CNN
 F 3 "~" H 5700 3700 50  0001 C CNN
 	1    5700 3700
